File: HSE42.kicad_sch (KiCad schematic)
At the start: 57 parts, among them J2 24PFPC, J6 CX90M, Q1 AO3400A, U1 SF32LB527UD6, U11 0524P, U2 PY25Q128HA-WXH-IR, U9 CH343P, Y1 48M

Commit message: update: 更新原理图
Parts:
- removed C53: 0.1u, Capacitor_SMD:C_0402_1005Metric, symbol Device:C
- added AE1: CA-C03, CrossAir ANT:CA-C03, symbol Device:Antenna_Shield
- added C16: 0.1u, symbol Device:C
- added C29: 1u, symbol Device:C
- added C30, C31: TBD, Capacitor_SMD:C_0402_1005Metric, symbol Device:C
- added C32: 22u, Capacitor_SMD:C_0603_1608Metric, symbol Device:C
- added C33, C36, C39, C45, C47: 0.1u, Capacitor_SMD:C_0402_1005Metric, symbol Device:C
- added C35, C37, C40: 330p, Capacitor_SMD:C_0402_1005Metric, symbol Device:C
- added C48, C54, C55: 1u, Capacitor_SMD:C_0402_1005Metric, symbol Device:C
- added D1: 1N4148, Diode_SMD:D_SOD-123F, symbol Device:D
- added D2: RED, LED_SMD:LED_0603_1608Metric, symbol Device:LED
- added FB1, FB2: 120R@100M, Inductor_SMD:L_0402_1005Metric, symbol Device:FerriteBead
- added J1, J3: GH1.25, Connector_JST:JST_GH_SM02B-GHS-TB_1x02-1MP_P1.25mm_Horizontal, symbol Connector_Generic_MountingPin:Conn_01x02_MountingPin
- added Q2: SI2305, Package_TO_SOT_SMD:SOT-23, symbol Device:Q_PMOS_GSD
- added R1: 1M, symbol Device:R
- added R12: 1M, Resistor_SMD:R_0402_1005Metric, symbol Device:R
- added R13, R14: 43.2k, Resistor_SMD:R_0402_1005Metric, symbol Device:R
- added R2: 82k, symbol Device:R
- added R21: 100k, Resistor_SMD:R_0402_1005Metric, symbol Device:R
- added R23, R26, R4: 10k, Resistor_SMD:R_0402_1005Metric, symbol Device:R
- added R3: TBD_R, Resistor_SMD:R_0402_1005Metric, symbol Device:R
- added R5: 0R, Resistor_SMD:R_0603_1608Metric, symbol Device:R
- added SW1, SW2, SW3: SW_Push, symbol Switch:SW_Push
- added U3: SHT40, Sensor_Humidity:Sensirion_DFN-4_1.5x1.5mm_P0.8mm_SHT4x_NoCentralPad, symbol Sensor_Humidity:SHT4x
- added U4: AW32901, My BGA:BGA-12_4x3_1.8x1.3mm, symbol OVP:AW329xx
- added U5: AW3512, Package_CSP:WLCSP-4_0.89x0.89mm_Layout2x2_P0.5mm, symbol Power_Management:AP22913CN4
- added U6: NS4150B, Package_SO:MSOP-8_3x3mm_P0.65mm, symbol Amplifier_Audio:LM4990MM
- added Y2: 32.768k, Crystal:Crystal_SMD_3215-2Pin_3.2x1.5mm, symbol Device:Crystal_Small
- R24, R25: value 100R -> 10k
Connections:
- net SF_D+ is gone; now on net KEY2: U1.65 (PA35)
- net SF_D- is gone; now on net KEY3: U1.64 (PA36)
- net +5V: now also C57.1, U9.3 (VDD5), U9.9 (VBUS), C29.1, D1.2 (A), Q2.1 (G), R21.1, R26.1, R5.2, U4.A2 (OUT), U4.A3 (OUT), U4.B2 (OUT)
- net DACN: now also C39.1
- net DACP: now also C36.1
- net EN: now also C45.2, R4.2, U5.B2 (ON)
- net GND: now also R24.2, R25.2, C16.2, C29.2, C30.2, C31.2, C35.2, C40.1, C47.2, C48.2, C54.2, C55.2, D2.1 (K), J1.1 (Pin_1), R2.2, R21.2, R23.2, U3.4 (VSS), U4.A1 (~{EN}), U4.A4 (GND), U4.B4 (GND), U4.C4 (GND), U5.B1 (GND), U6.7 (GND)
- net PA18: now also U9.4 (TXD); no longer R24.2
- net PA19: now also U9.5 (RXD); no longer R25.2
- net VBAT: now also J1.2 (Pin_2), Q2.3 (D)
- net VBUS: now also C16.1, R1.1, R5.1, U4.B3 (IN), U4.C2 (IN), U4.C3 (IN); no longer C57.1, U9.3 (VDD5), U9.9 (VBUS)
- net VCC: now also C32.1, C33.1, C55.1, U5.A1 (OUT), U6.6 (V+)
- net VDD33_2: now also C47.1, U3.3 (VDD)
- net VSYS: now also SW1.2, SW2.2, SW3.2
- net at U9.13 (RTS): now also C45.1
- net KEY2: now reaches R24.1
- net KEY2: now also SW2.1; no longer U9.4 (TXD)
- net KEY3: now reaches R25.1
- net KEY3: now also SW3.1; no longer U9.5 (RXD)
- net at U1.53 (ANT): now also C30.1, R3.1
- net DISPLAY_D10: no longer names the net of U1.60 (PA40)
- net DISPLAY_D11: no longer names the net of U1.59 (PA41)
- net DISPLAY_D12: no longer names the net of U1.58 (PA42)
- net DISPLAY_D13: no longer names the net of U1.57 (PA43)
- net DISPLAY_D6: no longer names the net of U1.44 (PA7)
- net DISPLAY_D7: no longer names the net of U1.43 (PA8)
- net DISPLAY_D8: no longer names the net of U1.63 (PA37)
- net DISPLAY_D9: no longer names the net of U1.61 (PA39)
- net PA10: no longer names the net of U1.35 (PA10)
- net PA11: no longer names the net of U1.34 (PA11)
- net PA20: no longer names the net of U1.25 (PA20)
- net PA22: no longer names the net of U1.11 (PA22)
- net PA22: now also Y2.2
- net PA23: no longer names the net of U1.10 (PA23)
- net PA23: now also Y2.1
- net PA24: no longer names the net of U1.9 (PA24)
- net PA25: no longer names the net of U1.8 (PA25)
- net PA26: no longer names the net of U1.7 (PA26)
- net PA27: no longer names the net of U1.6 (PA27)
- net PA28: no longer names the net of U1.5 (PA28)
- net PA29: no longer names the net of U1.4 (PA29)
- net PA30: no longer names the net of U1.3 (PA30)
- net PA31: no longer names the net of U1.2 (PA31)
- net PA32: no longer names the net of U1.1 (PA32)
- net PA33: no longer names the net of U1.67 (PA33)
- net PA34 renamed KEY1
- net KEY1: now also R23.1, SW1.1
- net PA38: no longer names the net of U1.62 (PA38)
- net PA44: no longer names the net of U1.56 (PA44)
- net PA9: no longer names the net of U1.42 (PA9)
- new net: R1.2, R2.1, U4.C1 (OVLO)
- new net: AE1.1 (A), C31.1, R3.2
- new net: C37.2, C40.2, FB2.2, J3.1 (Pin_1)
- new net: C54.1, D1.1 (K), Q2.2 (S), R4.1, U5.A2 (IN)
- new net: FB1.1, U6.8
- new net: C35.1, C37.1, FB1.2, J3.2 (Pin_2)
- new net: C39.2, R14.1
- new net: D2.2 (A), R26.2
- new net: R14.2, U6.4 (-)
- new net: C36.2, R13.1
- new net: R13.2, U6.3 (+)
- new net: C48.1, U6.2 (BYP)
- new net: FB2.1, U6.5
- new net GNDA: C32.2, C33.2, R12.2
- new net IIC_SCL: U3.2 (SCL)
- new net IIC_SDA: U3.1 (SDA)
- new net PA_EN: R12.1, U6.1 (~{SHDN})
- no-connect marks 12 -> 16
Other:
- moved on the sheet: C1, C10, C11, C12, C13, C14, C15, C17, C18, C19, C2, C20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
